File: FloppyKBD/FD00/Kicad/FD00.kicad_sch (KiCad schematic)
At the start: 30 parts, among them SW1 SW_PUSH, SW10 SW_PUSH, SW11 SW_PUSH, SW12 SW_PUSH, SW13 SW_PUSH, SW14 SW_PUSH, SW15 SW_PUSH, SW2 SW_PUSH, SW3 SW_PUSH, SW4 SW_PUSH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

Commit message: first commit
Parts:
- D1, D10, D11, D12, D13, D14, D2, D3, D4, D5, D6, D7, D8, D9: symbol Simulation_SPICE:DIODE -> Device:D
Changed lines of the file:
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@@
     )
   )
-  (symbol (lib_id "Simulation_SPICE:DIODE") (at 116.84 156.21 270) (unit 1)
+  (symbol (lib_id "Device:D") (at 116.84 156.21 270) (unit 1)
     (in_bom yes) (on_board yes) (fields_autoplaced)
     (property "Reference" "D2" (id 0) (at 119.38 154.9399 90)
@@
     (pin "2")
   )
-  (symbol (lib_id "Simulation_SPICE:DIODE") (at 91.44 232.41 270) (unit 1)
+  (symbol (lib_id "Device:D") (at 91.44 232.41 270) (unit 1)
     (in_bom yes) (on_board yes) (fields_autoplaced)
     (property "Reference" "D12" (id 0) (at 93.98 231.1399 90)
@@
     (pin "2")
   )
-  (symbol (lib_id "Simulation_SPICE:DIODE") (at 116.84 181.61 270) (unit 1)
+  (symbol (lib_id "Device:D") (at 116.84 181.61 270) (unit 1)
     (in_bom yes) (on_board yes) (fields_autoplaced)
     (property "Reference" "D5" (id 0) (at 119.38 180.3399 90)
@@
     (pin "2")
   )
-  (symbol (lib_id "Simulation_SPICE:DIODE") (at 142.24 232.41 270) (unit 1)
+  (symbol (lib_id "Device:D") (at 142.24 232.41 270) (unit 1)
     (in_bom yes) (on_board yes) (fields_autoplaced)
     (property "Reference" "D14" (id 0) (at 144.78 231.1399 90)
@@
     (pin "2")
   )
-  (symbol (lib_id "Simulation_SPICE:DIODE") (at 142.24 156.21 270) (unit 1)
+  (symbol (lib_id "Device:D") (at 142.24 156.21 270) (unit 1)
     (in_bom yes) (on_board yes) (fields_autoplaced)
     (property "Reference" "D3" (id 0) (at 144.78 154.9399 90)
@@
     (pin "2")
   )
-  (symbol (lib_id "Simulation_SPICE:DIODE") (at 116.84 232.41 270) (unit 1)
+  (symbol (lib_id "Device:D") (at 116.84 232.41 270) (unit 1)
     (in_bom yes) (on_board yes) (fields_autoplaced)
     (property "Reference" "D13" (id 0) (at 119.38 231.1399 90)
@@
     (pin "1")
   )
-  (symbol (lib_id "Simulation_SPICE:DIODE") (at 142.24 207.01 270) (unit 1)
+  (symbol (lib_id "Device:D") (at 142.24 207.01 270) (unit 1)
     (in_bom yes) (on_board yes) (fields_autoplaced)
     (property "Reference" "D10" (id 0) (at 144.78 205.7399 90)
@@
     (pin "9")
   )
-  (symbol (lib_id "Simulation_SPICE:DIODE") (at 66.04 207.01 270) (unit 1)
+  (symbol (lib_id "Device:D") (at 66.04 207.01 270) (unit 1)
     (in_bom yes) (on_board yes) (fields_autoplaced)
     (property "Reference" "D7" (id 0) (at 68.58 205.7399 90)
@@
     (pin "2")
   )
-  (symbol (lib_id "Simulation_SPICE:DIODE") (at 91.44 156.21 270) (unit 1)
+  (symbol (lib_id "Device:D") (at 91.44 156.21 270) (unit 1)
     (in_bom yes) (on_board yes) (fields_autoplaced)
     (property "Reference" "D1" (id 0) (at 93.98 154.9399 90)
@@
     (pin "1")
   )
-  (symbol (lib_id "Simulation_SPICE:DIODE") (at 91.44 181.61 270) (unit 1)
+  (symbol (lib_id "Device:D") (at 91.44 181.61 270) (unit 1)
     (in_bom yes) (on_board yes) (fields_autoplaced)
     (property "Reference" "D4" (id 0) (at 93.98 180.3399 90)
@@
     (pin "1")
   )
-  (symbol (lib_id "Simulation_SPICE:DIODE") (at 142.24 181.61 270) (unit 1)
+  (symbol (lib_id "Device:D") (at 142.24 181.61 270) (unit 1)
     (in_bom yes) (on_board yes) (fields_autoplaced)
     (property "Reference" "D6" (id 0) (at 144.78 180.3399 90)
@@
     (pin "2")
   )
-  (symbol (lib_id "Simulation_SPICE:DIODE") (at 66.04 232.41 270) (unit 1)
+  (symbol (lib_id "Device:D") (at 66.04 232.41 270) (unit 1)
     (in_bom yes) (on_board yes) (fields_autoplaced)
     (property "Reference" "D11" (id 0) (at 68.58 231.1399 90)
@@
     (pin "1")
   )
-  (symbol (lib_id "Simulation_SPICE:DIODE") (at 116.84 207.01 270) (unit 1)
+  (symbol (lib_id "Device:D") (at 116.84 207.01 270) (unit 1)
     (in_bom yes) (on_board yes) (fields_autoplaced)
     (property "Reference" "D9" (id 0) (at 119.38 205.7399 90)
@@
     (pin "1")
   )
-  (symbol (lib_id "Simulation_SPICE:DIODE") (at 91.44 207.01 270) (unit 1)
+  (symbol (lib_id "Device:D") (at 91.44 207.01 270) (unit 1)
     (in_bom yes) (on_board yes) (fields_autoplaced)
     (property "Reference" "D8" (id 0) (at 93.98 205.7399 90)
